File: usbc-i2c.kicad_pcb (KiCad board)
At the start: 2 copper layers, 50 x 30 mm, 14 parts, among them J1 HRO TYPE-C-31-M-12, J2 I2C, U1 AMS1117-3.3

Commit message: chore(layout): extract_layout round-trip — captures hand-routed I²C fan-out
User routed +3V3 / SDA / SCL / N_D1 in KiCad GUI; extract_layout pulled
the resulting 44 tracks (was 20) into layout.py via the four-marker-block
format. 9 of 10 unconnected items resolved.

Round-trip note: rebuilding from layout.py produces 7 violations + 3
unconnected, vs the saved KiCad PCB at 29 + 1. The delta:
  - zone clearance violations vanish on rebuild because build_pcb
    creates but doesn't auto-fill zones (KiCad fills on edit, so the
    saved PCB shows real-copper clearance checks)
  - 2 connections KiCad auto-snapped (track endpoints near but not
    exactly on pads) get lost — the round-trip captures the segment
    geometry literally, not the snap relationship

Both deltas are inherent to "code-as-source" PCB design: the GUI does
heuristic resolution that text round-trip can't replicate. Acceptable
for the regenerate-from-text promise; future work could add a snap-to-
nearest-pad pass in build_pcb to close the 2-pad gap.

Co-Authored-By: Claude Opus 4.7 (1M context) <noreply@anthropic.com>
Routing:
- net +3V3: track 0.00 -> 45.5 mm
- net SDA: track 0.00 -> 21.6 mm
- net SCL: track 0.00 -> 15.3 mm
- net N_D1: track 0.00 -> 5.40 mm
